File: deck_boardv1.2.kicad_sch (KiCad schematic)
At the start: 25 parts, among them J1 D-Sub 15 Pin Male Socket, U1 Raspberry Pi Zero 2 W, U2 LT8610AC, U3 XBP24-Z7SIT-004, U4 ADP7158ARDZ-3.3-R7

Commit message: PCB is mostly laid out, routing is WIP
Parts:
- removed J1: D-Sub 15 Pin Male Socket, Connector_Dsub:DSUB-15-HD_Socket_Vertical_P2.29x1.98mm_MountingHoles, symbol Connector:DA15_Pins
- added C14, C17: 47µF, Capacitor_SMD:C_0603_1608Metric, symbol Device:C
- added C15: 47pF, Capacitor_SMD:C_0603_1608Metric, symbol Device:C
- added C16: 1µF, Capacitor_SMD:C_0603_1608Metric, symbol Device:C
- added J1: 430450800, HarnessDeck:MOLEX_430450800, symbol 430450800:430450800
- C7: value 100µF -> 47µF
- L3: value 10µH -> 4.7µH
- R15: value 110k -> 60.4kΩ
- R16: value 191k -> 100kΩ
- R17: value 1M -> 412kΩ
- R18: value 100k -> 100kΩ
- R19: value 1 kohm -> 1 kΩ
- R20: value 4.7/10 kohm -> 10 kΩ
- U3: value XBP24-Z7SIT-004 -> DIGI XBee-PRO 900HP RF Module (S3B); footprint XBee:XBP24-Z7SIT-004 -> XBee:DIP2200W51P200L3294H279Q20P
- U4: value ADP7158ARDZ-3.3-R7 -> ADP7159
Connections:
- net 28v_inhibit/28v_IN: now also J1.1
- net 3V3: now also C15.1, C16.1; no longer U3.14 (VREF)
- net 5V_Pi: now also C14.2, C17.1
- net GND: now also U1.6 (GND_6), U3.14 (VREF), C14.1, C15.2, C16.2, C17.2, J1.2, J1.4, J1.6; no longer C5.2, R16.2, R17.1, U2.16 (FB)
- net TE_1: now also U1.11 (GPIO17-Camera_Select), J1.3
- net TE_2: now also J1.5
- new net: C5.2, R16.2, R17.1, U2.16 (FB)
Other:
- moved on the sheet: C10, C11, C12, C2, C3, C5, C6, C7, C8, D6, L3, R15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
