File: 28v_inhibit.kicad_sch (KiCad schematic)
At the start: 19 parts, among them Q1 Q_PMOS_GSD, Q2 Q_PMOS_GSD, Q3 NMOS, SW1 SAFE_switch, SW2 G-switch

Commit message: Edits to board post PDR.
Parts:
- removed SW2: G-switch, symbol Switch:SW_SPST
- added R22: 10 kohm, symbol Device:R_US
- R5: value R (1 kohm) -> 1 kohm
- R6: value R (100 kohm) -> 100 kohm
Connections:
- net 28V_Post_Inhibit: now also R22.2
- net GND: now also D4.1 (K)
- net at SW1.2 (B): now also R5.2, R6.2
- net at D4.2 (A): now also R22.1
Other:
- note added: "LED is on when the 1st inhibit chain and SAFE/ARM switch is passed."
- note added: "logical power gate. DECK only turns ON when RBF pin is pulled."
- note removed: "acceleration-triggered contact?"
- note removed: "logical power gate. DECK only turns ON when both armed manually and deployed."
- moved on the sheet: D3, D4, Q2, Q3, R3, R4, R5, R6, SW1

Commit message: Updated files and include work done for PCB
Parts:
- C1: footprint (none) -> Capacitor_SMD:C_0603_1608Metric
- D2, D3: footprint (none) -> Diode_SMD:D_SOD-123
- D4: footprint (none) -> LED_SMD:LED_0603_1608Metric
- F1: footprint (none) -> Fuse:Fuse_1206_3216Metric
- L1, L2: footprint (none) -> Inductor_SMD:L_0805_2012Metric
- Q1, Q2: footprint (none) -> Package_TO_SOT_SMD:SOT-223-3_TabPin2
- Q3: footprint (none) -> Package_TO_SOT_SMD:SOT-23
- R1, R3: value R (100 ohm) -> 100 ohm; footprint (none) -> Resistor_SMD:R_0201_0603Metric
- R2, R4: value R (100 kohm) -> 100 kohm; footprint (none) -> Resistor_SMD:R_0201_0603Metric
- R22, R5, R6: footprint (none) -> Resistor_SMD:R_0201_0603Metric
- SW1: footprint (none) -> Connector_PinHeader_2.54mm:PinHeader_1x02_P2.54mm_Vertical
Changed lines of the file:
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@@
 			)
 		)
-		(property "Value" "R (100 ohm)"
+		(property "Value" "100 ohm"
 			(at 60.96 107.9499 0)
 			(effects
@@
 			)
 		)
-		(property "Footprint" ""
+		(property "Footprint" "Resistor_SMD:R_0201_0603Metric"
 			(at 59.436 106.934 90)
 			(effects
@@
 			)
 		)
-		(property "Footprint" ""
+		(property "Footprint" "Diode_SMD:D_SOD-123"
 			(at 64.77 52.07 0)
 			(effects
@@
 			)
 		)
-		(property "Footprint" ""
+		(property "Footprint" "Connector_PinHeader_2.54mm:PinHeader_1x02_P2.54mm_Vertical"
 			(at 66.04 140.97 0)
 			(effects
@@
 			)
 		)
-		(property "Value" "R (100 kohm)"
+		(property "Value" "100 kohm"
 			(at 72.39 58.4199 0)
 			(effects
@@
 			)
 		)
-		(property "Footprint" ""
+		(property "Footprint" "Resistor_SMD:R_0201_0603Metric"
 			(at 70.866 57.404 90)
 			(effects
@@
 			)
 		)
-		(property "Footprint" ""
+		(property "Footprint" "Capacitor_SMD:C_0603_1608Metric"
 			(at 93.6752 49.53 0)
 			(effects
@@
 			)
 		)
-		(property "Footprint" ""
+		(property "Footprint" "Resistor_SMD:R_0201_0603Metric"
 			(at 103.886 125.984 90)
 			(effects
@@
 			)
 		)
-		(property "Footprint" ""
+		(property "Footprint" "Package_TO_SOT_SMD:SOT-223-3_TabPin2"
 			(at 67.31 33.02 0)
 			(effects
@@
 			)
 		)
-		(property "Footprint" ""
+		(property "Footprint" "Inductor_SMD:L_0805_2012Metric"
 			(at 101.6 35.56 0)
 			(effects
@@
 			)
 		)
-		(property "Footprint" ""
+		(property "Footprint" "Diode_SMD:D_SOD-123"
 			(at 53.34 111.76 0)
 			(effects
@@
 			)
 		)
-		(property "Footprint" ""
+		(property "Footprint" "Inductor_SMD:L_0805_2012Metric"
 			(at 82.55 35.56 0)
 			(effects
@@
 			)
 		)
-		(property "Footprint" ""
+		(property "Footprint" "LED_SMD:LED_0603_1608Metric"
 			(at 99.06 83.82 0)
 			(effects
@@
 			)
 		)
-		(property "Value" "R (100 kohm)"
+		(property "Value" "100 kohm"
 			(at 60.96 118.1099 0)
 			(effects
@@
 			)
 		)
-		(property "Footprint" ""
+		(property "Footprint" "Resistor_SMD:R_0201_0603Metric"
 			(at 59.436 117.094 90)
 			(effects
@@
 			)
 		)
-		(property "Footprint" ""
+		(property "Footprint" "Resistor_SMD:R_0201_0603Metric"
 			(at 87.376 125.984 90)
 			(effects
@@
 			)
 		)
-		(property "Footprint" ""
+		(property "Footprint" "Package_TO_SOT_SMD:SOT-223-3_TabPin2"
 			(at 55.88 91.44 0)
 			(effects
@@
 			)
 		)
-		(property "Footprint" ""
+		(property "Footprint" "Package_TO_SOT_SMD:SOT-23"
 			(at 83.82 109.22 0)
 			(effects
@@
 			)
 		)
-		(property "Footprint" ""
+		(property "Footprint" "Fuse:Fuse_1206_3216Metric"
 			(at 44.45 37.338 90)
 			(effects
@@
 			)
 		)
-		(property "Footprint" ""
+		(property "Footprint" "Resistor_SMD:R_0201_0603Metric"
 			(at 83.566 84.836 90)
 			(effects
@@
 			)
 		)
-		(property "Value" "R (100 ohm)"
+		(property "Value" "100 ohm"
 			(at 72.39 48.2599 0)
 			(effects
@@
 			)
 		)
-		(property "Footprint" ""
+		(property "Footprint" "Resistor_SMD:R_0201_0603Metric"
 			(at 70.866 47.244 90)
 			(effects

Commit message: PCB is mostly laid out, routing is WIP
Parts:
- added D9: BZT52B12, Diode_SMD:D_SOD-123, symbol Device:D_Zener
- C1: value C -> 22 µF
- D1: value SMAJ33A -> SMAJ36A
- D2, D3: value D_Zener -> BZT52B12
- F1: value Fuse -> 045101.5
- L1, L2: value L -> 2.2µH
- Q1, Q2: value Q_PMOS_GSD -> FQPF27P06
- Q3: value NMOS -> 2N7000
- R1, R3: value 100 ohm -> 100Ω
- R2, R4, R6: value 100 kohm -> 100kΩ
- R22: value 10 kohm -> 10kΩ
- R5: value 1 kohm -> 10kΩ
Connections:
- net GND: now also D9.2 (A)
- net at R5.2, R6.2, SW1.2 (B): now also D9.1 (K)
Other:
- note added: "manual arming switch RBF PIN"
- note removed: "manual arming switch"
Changed lines of the file:
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@@
 		)
 	)
-	(text "manual arming switch\n"
-		(exclude_from_sim no)
-		(at 67.31 144.526 0)
+	(text "manual arming switch\nRBF PIN\n"
+		(exclude_from_sim no)
+		(at 66.548 145.288 0)
 		(effects
 			(font
@@
 	)
 	(junction
+		(at 96.52 132.08)
+		(diameter 0)
+		(color 0 0 0 0)
+	)
+	(junction
 		(at 52.07 35.56)
 		(diameter 0)
@@
 	)
 	(junction
+		(at 96.52 111.76)
+		(diameter 0)
+		(color 0 0 0 0)
+	)
+	(junction
 		(at 44.45 124.46)
 		(diameter 0)
@@
 	(wire
 		(pts
-			(xy 91.44 111.76) (xy 102.87 111.76)
+			(xy 91.44 111.76) (xy 96.52 111.76)
 		)
 		(stroke
@@
 	(wire
 		(pts
+			(xy 96.52 129.54) (xy 96.52 132.08)
+		)
+		(stroke
+			(width 0)
+			(type default)
+		)
+	)
+	(wire
+		(pts
 			(xy 69.85 50.8) (xy 69.85 52.07)
 		)
@@
 	(wire
 		(pts
-			(xy 86.36 132.08) (xy 102.87 132.08)
+			(xy 86.36 132.08) (xy 96.52 132.08)
 		)
 		(stroke
@@
 	(wire
 		(pts
+			(xy 96.52 111.76) (xy 96.52 121.92)
+		)
+		(stroke
+			(width 0)
+			(type default)
+		)
+	)
+	(wire
+		(pts
 			(xy 92.71 49.53) (xy 92.71 62.23)
 		)
@@
 	(wire
 		(pts
+			(xy 96.52 132.08) (xy 102.87 132.08)
+		)
+		(stroke
+			(width 0)
+			(type default)
+		)
+	)
+	(wire
+		(pts
 			(xy 52.07 35.56) (xy 52.07 41.91)
 		)
@@
 		(pts
 			(xy 69.85 62.23) (xy 69.85 60.96)
+		)
+		(stroke
+			(width 0)
+			(type default)
+		)
+	)
+	(wire
+		(pts
+			(xy 96.52 111.76) (xy 102.87 111.76)
 		)
 		(stroke
@@
 			)
 		)
-		(property "Value" "100 ohm"
+		(property "Value" "100Ω"
 			(at 60.96 107.9499 0)
 			(effects
@@
 			)
 		)
-		(property "Value" "D_Zener"
-			(at 59.944 55.626 0)
+		(property "Value" "BZT52B12"
+			(at 58.166 55.626 0)
 			(effects
 				(font
@@
 			)
 		)
-		(property "Value" "100 kohm"
+		(property "Value" "100kΩ"
 			(at 72.39 58.4199 0)
 			(effects
@@
 			)
 		)
-		(property "Value" "C"
+		(property "Value" "22 µF"
 			(at 96.52 46.9899 0)
 			(effects
@@
 			)
 		)
-		(property "Value" "SMAJ33A"
+		(property "Value" "SMAJ36A"
 			(at 45.72 44.958 90)
 			(effects
@@
 			)
 		)
-		(property "Value" "100 kohm"
+		(property "Value" "100kΩ"
 			(at 105.41 126.9999 0)
 			(effects
@@
 			)
 		)
-		(property "Value" "Q_PMOS_GSD"
+		(property "Value" "FQPF27P06"
 			(at 69.85 31.75 90)
 			(effects
@@
 			)
 		)
-		(property "Value" "L"
+		(property "Value" "2.2µH"
 			(at 101.6 33.02 90)
 			(effects
@@
 			)
 		)
-		(property "Value" "D_Zener"
+		(property "Value" "BZT52B12"
 			(at 51.054 108.458 0)
 			(effects
@@
 			)
 		)
-		(property "Value" "L"
+		(property "Value" "2.2µH"
 			(at 82.55 33.02 90)
 			(effects
@@
 			)
 		)
-		(property "Value" "100 kohm"
+		(property "Value" "100kΩ"
 			(at 60.96 118.1099 0)
 			(effects
@@
 		(on_board yes)
 		(dnp no)
-		(fields_autoplaced yes)
 		(property "Reference" "R5"
-			(at 88.9 124.4599 0)
+			(at 78.994 124.206 0)
 			(effects
 				(font
@@
 			)
 		)
-		(property "Value" "1 kohm"
-			(at 88.9 126.9999 0)
+		(property "Value" "10kΩ"
+			(at 78.994 126.746 0)
 			(effects
 				(font
@@
 			)
 		)
-		(property "Value" "Q_PMOS_GSD"
+		(property "Value" "FQPF27P06"
 			(at 58.42 90.17 90)
 			(effects
@@
 				(path "/0dd6c749-d328-44a2-b3d4-206fc5899db9/1f8cf09f-ba90-4e4f-a442-1634942ef321"
 					(reference "Q2")
+					(unit 1)
+				)
+			)
+		)
+	)
+	(symbol
+		(lib_id "Device:D_Zener")
+		(at 96.52 125.73 90)
+		(unit 1)
+		(exclude_from_sim no)
+		(in_bom yes)
+		(on_board yes)
+		(dnp no)
+		(property "Reference" "D9"
+			(at 92.456 120.396 90)
+			(effects
+				(font
+					(size 1.27 1.27)
+				)
+			)
+		)
+		(property "Value" "BZT52B12"
+			(at 92.71 122.682 90)
+			(effects
+				(font
+					(size 1.27 1.27)
+				)
+			)
+		)
+		(property "Footprint" "Diode_SMD:D_SOD-123"
+			(at 96.52 125.73 0)
+			(effects
+				(font
+					(size 1.27 1.27)
+				)
+				(hide yes)
+			)
+		)
+		(property "Datasheet" "~"
+			(at 96.52 125.73 0)
+			(effects
+				(font
+					(size 1.27 1.27)
+				)
+				(hide yes)
+			)
+		)
+		(property "Description" "Zener diode"
+			(at 96.52 125.73 0)
+			(effects
+				(font
+					(size 1.27 1.27)
+				)
+				(hide yes)
+			)
+		)
+		(pin "1"
+		)
+		(pin "2"
+		)
+		(instances
+			(project "deck_boardv1.1"
+				(path "/0dd6c749-d328-44a2-b3d4-206fc5899db9/1f8cf09f-ba90-4e4f-a442-1634942ef321"
+					(reference "D9")
 					(unit 1)
 				)
@@
 			)
 		)
-		(property "Value" "NMOS"
+		(property "Value" "2N7000"
 			(at 86.36 107.95 90)
 			(effects
@@
 			)
 		)
-		(property "Value" "Fuse"
-			(at 46.482 32.766 90)
+		(property "Value" "045101.5"
+			(at 48.006 33.02 90)
 			(effects
 				(font
@@
 			)
 		)
-		(property "Value" "10 kohm"
+		(property "Value" "10kΩ"
 			(at 83.82 80.01 90)
 			(effects
@@
 			)
 		)
-		(property "Value" "100 ohm"
+		(property "Value" "100Ω"
 			(at 72.39 48.2599 0)
 			(effects

Commit message: Made changes to schematic
Parts:
- removed D1: SMAJ36A, Diode_SMD:D_SMA, symbol Diode:SMAJ33A
- removed D2, D3, D9: BZT52B12, Diode_SMD:D_SOD-123, symbol Device:D_Zener
- removed F1: 045101.5, Fuse:Fuse_1206_3216Metric, symbol Device:Fuse
- removed L1, L2: 2.2µH, Inductor_SMD:L_0805_2012Metric, symbol Device:L
- removed Q1, Q2: FQPF27P06, Package_TO_SOT_SMD:SOT-223-3_TabPin2, symbol Transistor_FET:Q_PMOS_GSD
- removed Q3: 2N7000, Package_TO_SOT_SMD:SOT-23, symbol Simulation_SPICE:NMOS
- removed R2, R4, R6: 100kΩ, Resistor_SMD:R_0201_0603Metric, symbol Device:R_US
- removed R22, R5: 10kΩ, Resistor_SMD:R_0201_0603Metric, symbol Device:R_US
- removed R3: 100Ω, Resistor_SMD:R_0201_0603Metric, symbol Device:R_US
- removed SW1: SAFE_switch, Connector_PinHeader_2.54mm:PinHeader_1x02_P2.54mm_Vertical, symbol Switch:SW_SPST
- added D2: STPS5H100B, STPS5H100B:DPAK, symbol STPS5H100B:STPS5H100B
- added SW1: Inhibit Switch (SS-5GL?), symbol Switch:SW_Push_SPDT
- C1: value 22 µF -> 47 µF
- D4: value LED -> Red LED
- R1: value 100Ω -> 18kΩ
Connections:
- net 28V_Post_Inhibit: now also C1.1, R1.2, SW1.3 (C)
- net 28v_IN: now also D2.3
- net at R1.1: now also D4.2 (A)
- new net: D2.2, SW1.2 (B)
- no-connect marks 0 -> 1
Other:
- note added: "LED is on when switch is passed."
- note removed: "Keeps DECK from drawing current until ground testing safety rules are met. Protects against voltage reversal or spikes from 28v supply. -always ON for correct polarity -blocks reverse voltage"
- note removed: "LED is on when the 1st inhibit chain and SAFE/ARM switch is passed."
- note removed: "gate bias"
- note removed: "gate clamp"
- note removed: "logical power gate. DECK only turns ON when RBF pin is pulled."
- note removed: "low-pass filter"
- note removed: "manual arming switch RBF PIN"
- note removed: "protects DECK from internal shorts"
- note removed: "pull-down"
- note removed: "pull-up; keeps Q2 OFF by default"
- note removed: "pulls Q2 gate low when SAFE + G-switch closed"
- note removed: "when polarity correct, gate-source goes neg. turns ON. if polarity is reversed, turns OFF."
- moved on the sheet: D4
