File: inhibit_2.kicad_sch (KiCad schematic)
At the start: 4 parts, among them SW3 SAFE_switch, SW4 G-switch

Commit message: Edits to board post PDR.
Parts:
- removed SW4: G-switch, symbol Switch:SW_SPST
Connections:
- net ENABLE: now also SW3.2 (B)
Other:
- note added: "RBF pin that will stay in for ground testing, must be removed before mission."
- note removed: "TE_2 is a 28v line?"
- note removed: "might not need these here?"
- moved on the sheet: R7, R9, SW3
Changed lines of the file:
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@@
 	(generator_version "9.0")
 	(paper "A4")
-	(text "might not need these here?"
-		(exclude_from_sim no)
-		(at 73.914 72.644 0)
-		(effects
-			(font
-				(size 0.762 0.762)
+	(text "RBF pin that will stay in\nfor ground testing, must\nbe removed before mission."
+		(exclude_from_sim no)
+		(at 54.864 72.644 0)
+		(effects
+			(font
+				(size 1.27 1.27)
 			)
 		)
@@
 	(text "keeps DECK powered while preventing burn-wire \nfrom firing until TE_2 is achieved.\n"
 		(exclude_from_sim no)
-		(at 112.522 67.056 0)
+		(at 85.09 67.31 0)
 		(effects
 			(font
@@
 		)
 	)
-	(text "TE_2 is a 28v line?"
-		(exclude_from_sim no)
-		(at 40.132 58.928 0)
-		(effects
-			(font
-				(size 1.27 1.27)
-			)
-		)
-	)
 	(junction
-		(at 57.15 54.61)
+		(at 46.99 53.34)
 		(diameter 0)
 		(color 0 0 0 0)
@@
 	(wire
 		(pts
-			(xy 57.15 68.58) (xy 59.69 68.58)
-		)
-		(stroke
-			(width 0)
-			(type default)
-		)
-	)
-	(wire
-		(pts
-			(xy 68.58 54.61) (xy 77.47 54.61)
-		)
-		(stroke
-			(width 0)
-			(type default)
-		)
-	)
-	(wire
-		(pts
-			(xy 57.15 68.58) (xy 57.15 54.61)
-		)
-		(stroke
-			(width 0)
-			(type default)
-		)
-	)
-	(wire
-		(pts
-			(xy 54.61 54.61) (xy 57.15 54.61)
-		)
-		(stroke
-			(width 0)
-			(type default)
-		)
-	)
-	(wire
-		(pts
-			(xy 88.9 68.58) (xy 97.79 68.58)
-		)
-		(stroke
-			(width 0)
-			(type default)
-		)
-	)
-	(wire
-		(pts
-			(xy 41.91 54.61) (xy 46.99 54.61)
-		)
-		(stroke
-			(width 0)
-			(type default)
-		)
-	)
-	(wire
-		(pts
-			(xy 57.15 54.61) (xy 60.96 54.61)
-		)
-		(stroke
-			(width 0)
-			(type default)
-		)
-	)
-	(wire
-		(pts
-			(xy 69.85 68.58) (xy 78.74 68.58)
+			(xy 46.99 67.31) (xy 49.53 67.31)
+		)
+		(stroke
+			(width 0)
+			(type default)
+		)
+	)
+	(wire
+		(pts
+			(xy 58.42 53.34) (xy 67.31 53.34)
+		)
+		(stroke
+			(width 0)
+			(type default)
+		)
+	)
+	(wire
+		(pts
+			(xy 46.99 67.31) (xy 46.99 53.34)
+		)
+		(stroke
+			(width 0)
+			(type default)
+		)
+	)
+	(wire
+		(pts
+			(xy 44.45 53.34) (xy 46.99 53.34)
+		)
+		(stroke
+			(width 0)
+			(type default)
+		)
+	)
+	(wire
+		(pts
+			(xy 31.75 53.34) (xy 36.83 53.34)
+		)
+		(stroke
+			(width 0)
+			(type default)
+		)
+	)
+	(wire
+		(pts
+			(xy 46.99 53.34) (xy 50.8 53.34)
+		)
+		(stroke
+			(width 0)
+			(type default)
+		)
+	)
+	(wire
+		(pts
+			(xy 59.69 67.31) (xy 67.31 67.31)
 		)
 		(stroke
@@
 	(hierarchical_label "GND"
 		(shape input)
-		(at 77.47 54.61 0)
+		(at 67.31 53.34 0)
 		(effects
 			(font
@@
 	(hierarchical_label "TE_2"
 		(shape input)
-		(at 41.91 54.61 180)
+		(at 31.75 53.34 180)
 		(effects
 			(font
@@
 	(hierarchical_label "ENABLE"
 		(shape input)
-		(at 97.79 68.58 0)
+		(at 67.31 67.31 0)
 		(effects
 			(font
@@
 			)
 			(justify left)
-		)
-	)
-	(symbol
-		(lib_id "Switch:SW_SPST")
-		(at 83.82 68.58 0)
-		(unit 1)
-		(exclude_from_sim no)
-		(in_bom yes)
-		(on_board yes)
-		(dnp no)
-		(fields_autoplaced yes)
-		(property "Reference" "SW4"
-			(at 83.82 62.23 0)
-			(effects
-				(font
-					(size 1.27 1.27)
-				)
-			)
-		)
-		(property "Value" "G-switch"
-			(at 83.82 64.77 0)
-			(effects
-				(font
-					(size 1.27 1.27)
-				)
-			)
-		)
-		(property "Footprint" ""
-			(at 83.82 68.58 0)
-			(effects
-				(font
-					(size 1.27 1.27)
-				)
-				(hide yes)
-			)
-		)
-		(property "Datasheet" "~"
-			(at 83.82 68.58 0)
-			(effects
-				(font
-					(size 1.27 1.27)
-				)
-				(hide yes)
-			)
-		)
-		(property "Description" "Single Pole Single Throw (SPST) switch"
-			(at 83.82 68.58 0)
-			(effects
-				(font
-					(size 1.27 1.27)
-				)
-				(hide yes)
-			)
-		)
-		(pin "2"
-		)
-		(pin "1"
-		)
-		(instances
-			(project "deck_board"
-				(path "/0dd6c749-d328-44a2-b3d4-206fc5899db9/9dadea64-6056-4d58-9d6d-a980455d899a"
-					(reference "SW4")
-					(unit 1)
-				)
-			)
 		)
 	)
 	(symbol
 		(lib_id "Device:R_US")
-		(at 64.77 54.61 270)
+		(at 54.61 53.34 270)
 		(unit 1)
 		(exclude_from_sim no)
@@
 		(fields_autoplaced yes)
 		(property "Reference" "R9"
-			(at 64.77 48.26 90)
+			(at 54.61 46.99 90)
 			(effects
 				(font
@@
 		)
 		(property "Value" "R"
-			(at 64.77 50.8 90)
+			(at 54.61 49.53 90)
 			(effects
 				(font
@@
 		)
 		(property "Footprint" ""
-			(at 64.516 55.626 90)
+			(at 54.356 54.356 90)
 			(effects
 				(font
@@
 		)
 		(property "Datasheet" "~"
-			(at 64.77 54.61 0)
+			(at 54.61 53.34 0)
 			(effects
 				(font
@@
 		)
 		(property "Description" "Resistor, US symbol"
-			(at 64.77 54.61 0)
+			(at 54.61 53.34 0)
 			(effects
 				(font
@@
 	(symbol
 		(lib_id "Device:R_US")
-		(at 50.8 54.61 270)
+		(at 40.64 53.34 270)
 		(unit 1)
 		(exclude_from_sim no)
@@
 		(fields_autoplaced yes)
 		(property "Reference" "R7"
-			(at 50.8 48.26 90)
+			(at 40.64 46.99 90)
 			(effects
 				(font
@@
 		)
 		(property "Value" "R"
-			(at 50.8 50.8 90)
+			(at 40.64 49.53 90)
 			(effects
 				(font
@@
 		)
 		(property "Footprint" ""
-			(at 50.546 55.626 90)
+			(at 40.386 54.356 90)
 			(effects
 				(font
@@
 		)
 		(property "Datasheet" "~"
-			(at 50.8 54.61 0)
+			(at 40.64 53.34 0)
 			(effects
 				(font
@@
 		)
 		(property "Description" "Resistor, US symbol"
-			(at 50.8 54.61 0)
+			(at 40.64 53.34 0)
 			(effects
 				(font
@@
 	(symbol
 		(lib_id "Switch:SW_SPST")
-		(at 64.77 68.58 0)
+		(at 54.61 67.31 0)
 		(unit 1)
 		(exclude_from_sim no)
@@
 		(fields_autoplaced yes)
 		(property "Reference" "SW3"
-			(at 64.77 62.23 0)
+			(at 54.61 60.96 0)
 			(effects
 				(font
@@
 		)
 		(property "Value" "SAFE_switch"
-			(at 64.77 64.77 0)
+			(at 54.61 63.5 0)
 			(effects
 				(font
@@
 		)
 		(property "Footprint" ""
-			(at 64.77 68.58 0)
+			(at 54.61 67.31 0)
 			(effects
 				(font
@@
 		)
 		(property "Datasheet" "~"
-			(at 64.77 68.58 0)
+			(at 54.61 67.31 0)
 			(effects
 				(font
@@
 		)
 		(property "Description" "Single Pole Single Throw (SPST) switch"
-			(at 64.77 68.58 0)
-			(effects
-				(font
+			(at 54.61 67.31 0)
+			(effects
+				(font

Commit message: Updated files and include work done for PCB
Parts:
- R7, R9: footprint (none) -> Resistor_SMD:R_0201_0603Metric
- SW3: footprint (none) -> Connector_PinHeader_2.54mm:PinHeader_1x02_P2.54mm_Vertical
Changed lines of the file:
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@@
 			)
 		)
-		(property "Footprint" ""
+		(property "Footprint" "Resistor_SMD:R_0201_0603Metric"
 			(at 54.356 54.356 90)
 			(effects
@@
 			)
 		)
-		(property "Footprint" ""
+		(property "Footprint" "Resistor_SMD:R_0201_0603Metric"
 			(at 40.386 54.356 90)
 			(effects
@@
 			)
 		)
-		(property "Footprint" ""
+		(property "Footprint" "Connector_PinHeader_2.54mm:PinHeader_1x02_P2.54mm_Vertical"
 			(at 54.61 67.31 0)
 			(effects

Commit message: PCB is mostly laid out, routing is WIP
Parts:
- removed R9: R, Resistor_SMD:R_0201_0603Metric, symbol Device:R_US
- added D5: 3.6 V Zener, Diode_SMD:D_SOD-123, symbol Device:D_Zener
- added R23: 100kΩ, Resistor_SMD:R_0201_0603Metric, symbol Device:R_US
- R7: value R -> 10kΩ
Connections:
- net ENABLE: now also R7.1, SW3.1 (A), D5.1 (K), R23.1; no longer SW3.2 (B)
- net GND: now also SW3.2 (B), D5.2 (A), R23.2
Other:
- note added: "goes to burn-wire circuit"
- note added: "when pin is in, shorts to GND"
- moved on the sheet: R7, SW3

Commit message: Finished PCB, ready to print
Parts:
- SW3: footprint Connector_PinHeader_2.54mm:PinHeader_1x02_P2.54mm_Vertical -> Connector_PinHeader_2.54mm:PinHeader_1x01_P2.54mm_Vertical
Changed lines of the file:
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@@
 			)
 		)
-		(property "Footprint" "Connector_PinHeader_2.54mm:PinHeader_1x02_P2.54mm_Vertical"
+		(property "Footprint" "Connector_PinHeader_2.54mm:PinHeader_1x01_P2.54mm_Vertical"
 			(at 69.85 69.85 0)
 			(effects

Commit message: Made changes to schematic
Parts:
- removed D5: 3.6 V Zener, Diode_SMD:D_SOD-123, symbol Device:D_Zener
- removed R23: 100kΩ, Resistor_SMD:R_0201_0603Metric, symbol Device:R_US
- removed SW3: SAFE_switch, Connector_PinHeader_2.54mm:PinHeader_1x01_P2.54mm_Vertical, symbol Switch:SW_SPST
Other:
- note removed: "RBF pin that will stay in for ground testing, must be removed before mission."
- note removed: "goes to burn-wire circuit"
- note removed: "when pin is in, shorts to GND"
