File: burn_wire.kicad_sch (KiCad schematic)
At the start: 7 parts, among them J2 Conn_01x01_Pin, J3 Conn_01x01_Pin, Q3 NMOS

Commit message: Added labels to silkscreen.
Parts:
- D6: footprint LED_SMD:LED_0603_1608Metric -> LED_THT:LED_D3.0mm
Changed lines of the file:
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@@
 			)
 		)
-		(property "Footprint" "LED_SMD:LED_0603_1608Metric"
+		(property "Footprint" "LED_THT:LED_D3.0mm"
 			(at 109.22 49.53 0)
 			(effects
