File: _autosave-deck_boardv1.5.kicad_sch (KiCad schematic)
At the start: 51 parts, among them J1 430450800, J4 Conn_01x01_Pin, J5 Conn_01x01_Pin, J6 Conn_01x01_Pin, J7 Conn_01x01_Pin, Q1 MMBT3904, Q2 2N7002, SW1 Inhibit Switch (SS-5GL), SW2 Inhibit Switch (SS-5GL), U1 Raspberry Pi Zero 2 W, U2 LT8610AC, U3 DIGI XBee-PRO 900HP RF Module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, U4 ADP7158ARDZ-3.3-R7

Commit message: Fixed general issues with footprints.
Parts:
- L1: footprint Inductor_SMD:L_Vishay_IHLP-2525 -> Library:0630CDMCCDS-100MC
Changed lines of the file:
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@@
 			)
 		)
-		(property "Footprint" "Inductor_SMD:L_Vishay_IHLP-2525"
+		(property "Footprint" "Library:0630CDMCCDS-100MC"
 			(at 99.06 40.64 0)
 			(effects
